File: rat_board.sch (KiCad schematic (older format))
At the start: 52 parts, among them P1 FRONT_LEFT_IR, P2 SIDE_LEFT_IR, P3 SIDE_RIGHT_IR, P4 FRONT_RIGHT_IR, P5 LEFT_MOTOR, P6 RIGHT_MOTOR, P7 JTAG, P8 CONN_01X02, P9 CONN_01X04, SW1 SW_PUSH_SMALL_H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

Commit message: solved oscillator bug
Parts:
- removed ext1: R, Resistors_SMD:R_0603_HandSoldering, symbol R
Connections:
- net GND: now also C7.2, C9.2; no longer Y1.2, Y2.2
- net OSC32IN: now also Y1.1
- net OSC32OUT: now also Y1.2
- net OSCIN: now also Y2.1
- net OSCOUT: now also C8.1, Y2.2
Other:
- moved on the sheet: C10, C9, Y1, Y2
Changed lines of the file:
@@
 L Crystal Y2
 U 1 1 587900B3
-P 10750 3100
-F 0 "Y2" H 10750 3250 50  0000 C CNN
-F 1 "8MHz" V 10750 2850 50  0000 C CNN
-F 2 "Crystals:Crystal_HC50-U_Vertical" H 10750 3100 50  0001 C CNN
-F 3 "" H 10750 3100 50  0000 C CNN
-	1    10750 3100
+P 10050 3100
+F 0 "Y2" H 10050 3250 50  0000 C CNN
+F 1 "8MHz" V 10050 2850 50  0000 C CNN
+F 2 "Crystals:Crystal_HC50-U_Vertical" H 10050 3100 50  0001 C CNN
+F 3 "" H 10050 3100 50  0000 C CNN
+	1    10050 3100
 	0    1    1    0
 $EndComp
@@
 	0    -1   -1   0
 $EndComp
-$Comp
-L R ext1
-U 1 1 5879026F
-P 10100 3350
-F 0 "ext1" V 10180 3350 50  0000 C CNN
-F 1 "R" V 10100 3350 50  0000 C CNN
-F 2 "Resistors_SMD:R_0603_HandSoldering" V 10030 3350 50  0001 C CNN
-F 3 "" H 10100 3350 50  0000 C CNN
-	1    10100 3350
-	0    1    1    0
-$EndComp
 Text Label 9350 2850 0    60   ~ 0
 OSCIN
@@
 L C C9
 U 1 1 58790916
-P 10100 3850
-F 0 "C9" H 10125 3950 50  0000 L CNN
-F 1 "20p" H 10125 3750 50  0000 L CNN
-F 2 "Capacitors_SMD:C_0603_HandSoldering" H 10138 3700 50  0001 C CNN
-F 3 "" H 10100 3850 50  0000 C CNN
-	1    10100 3850
+P 10400 3850
+F 0 "C9" H 10425 3950 50  0000 L CNN
+F 1 "20p" H 10425 3750 50  0000 L CNN
+F 2 "Capacitors_SMD:C_0603_HandSoldering" H 10438 3700 50  0001 C CNN
+F 3 "" H 10400 3850 50  0000 C CNN
+	1    10400 3850
 	0    -1   -1   0
 $EndComp
@@
 L Crystal Y1
 U 1 1 5879091C
-P 10550 4100
-F 0 "Y1" H 10550 4250 50  0000 C CNN
-F 1 "32.768kHz" V 10550 3750 50  0000 C CNN
-F 2 "Crystals:Crystal_MC-156" H 10550 4100 50  0001 C CNN
-F 3 "" H 10550 4100 50  0000 C CNN
-	1    10550 4100
+P 10050 4100
+F 0 "Y1" H 10050 4250 50  0000 C CNN
+F 1 "32.768kHz" V 10050 3750 50  0000 C CNN
+F 2 "Crystals:Crystal_MC-156" H 10050 4100 50  0001 C CNN
+F 3 "" H 10050 4100 50  0000 C CNN
+	1    10050 4100
 	0    1    1    0
 $EndComp
@@
 L C C10
 U 1 1 58790922
-P 10100 4350
-F 0 "C10" H 10125 4450 50  0000 L CNN
-F 1 "20p" H 10125 4250 50  0000 L CNN
-F 2 "Capacitors_SMD:C_0603_HandSoldering" H 10138 4200 50  0001 C CNN
-F 3 "" H 10100 4350 50  0000 C CNN
-	1    10100 4350
+P 10400 4350
+F 0 "C10" H 10425 4450 50  0000 L CNN
+F 1 "20p" H 10425 4250 50  0000 L CNN
+F 2 "Capacitors_SMD:C_0603_HandSoldering" H 10438 4200 50  0001 C CNN
+F 3 "" H 10400 4350 50  0000 C CNN
+	1    10400 4350
 	0    -1   -1   0
 $EndComp
@@
 	6050 2300 5650 2300
 Wire Wire Line
-	9350 2850 10250 2850
-Wire Wire Line
-	9350 3350 9950 3350
-Wire Wire Line
-	9350 3850 9950 3850
-Wire Wire Line
-	9350 4350 9950 4350
-Wire Wire Line
-	10250 4350 10750 4350
-Wire Wire Line
-	10750 4350 10750 4400
-Wire Wire Line
-	10550 4250 10550 4350
-Connection ~ 10550 4350
-Wire Wire Line
-	10550 3950 10550 3850
-Wire Wire Line
-	10550 3850 10250 3850
-Wire Wire Line
-	10750 3250 10750 3450
+	9350 3350 10250 3350
+Wire Wire Line
+	9350 3850 10250 3850
+Wire Wire Line
+	9350 4350 10250 4350
+Wire Wire Line
+	10750 3850 10750 4400
+Wire Wire Line
+	10750 2850 10750 3450
 Wire Wire Line
 	10750 3350 10550 3350
@@
 Wire Wire Line
 	10550 2850 10750 2850
-Wire Wire Line
-	10750 2850 10750 2950
 Wire Wire Line
 	9500 1500 9500 1050
@@
 Wire Wire Line
 	850  950  850  3050
+Wire Wire Line
+	9350 2850 10250 2850
+Wire Wire Line
+	10550 3850 10750 3850
+Wire Wire Line
+	10550 4350 10750 4350
+Connection ~ 10750 4350
+Wire Wire Line
+	10050 3950 10050 3850
+Connection ~ 10050 3850
+Wire Wire Line
+	10050 4250 10050 4350
+Connection ~ 10050 4350
+Wire Wire Line
+	10050 2850 10050 2950
+Connection ~ 10050 2850
+Wire Wire Line
+	10050 3250 10050 3350
+Connection ~ 10050 3350
 $EndSCHEMATC
